File: eagle files/shift controller.sch (EAGLE design)
At the start: 36 parts, among them IC1 LM340S

Commit message: board stuff
Parts:
- renumbered U$10 to CHANNEL_A, U$11 to CHANNEL_C, U$9 to CHANNEL_B
Connections:
- removed net N$17: C8.2, IC1.GND@1, IC1.GND@2, U$2.GND
- net N$13: no longer C6.1
- net N$35: now also C6.1, C8.2, IC1.GND@1, IC1.GND@2, U$2.GND
- net N$44: now also U$1.PA04; no longer U$1.PB09
- net N$45: now also U$1.PA05; no longer U$1.PA04
- net N$46: now also U$1.PA06; no longer U$1.PA05
- net N$47: now also U$1.PA07; no longer U$1.PA06
Other:
- moved on the sheet: C5, L1, SV1, SV2
